Commit message: add foreman, update launch files

File: workspaces/franka/srdf/franka.srdf.xacro (robot description, xacro)
@@ -1,21 +1,20 @@
 <?xml version="1.0" encoding="UTF-8"?>
 <robot name="franka" xmlns:xacro="http://wiki.ros.org/xacro">
-    <xacro:arg name="arm_id" default="fr3"/>
+    <xacro:arg name="robot_prefix" default="fr3"/>
     <xacro:include filename="$(find franka_description)/robots/common/franka_arm.srdf.xacro"/>
     <xacro:franka_arm_srdf
-            arm_id="$(arg arm_id)"
+            robot_type="fr3"
             hand="false"
             ee_id=""
             no_prefix="false"
-            arm_prefix=""
-            tip_link="link8"/>
-    <group_state name="home" group="$(arg arm_id)_arm">
-        <joint name="$(arg arm_id)_joint1" value="0" />
-        <joint name="$(arg arm_id)_joint2" value="-0.785398163397" />
-        <joint name="$(arg arm_id)_joint3" value="0" />
-        <joint name="$(arg arm_id)_joint4" value="-2.35619449019" />
-        <joint name="$(arg arm_id)_joint5" value="0" />
-        <joint name="$(arg arm_id)_joint6" value="1.57079632679" />
-        <joint name="$(arg arm_id)_joint7" value="0.785398163397" />
+            arm_prefix="$(arg robot_prefix)"/>
+    <group_state name="home" group="$(arg robot_prefix)_arm">
+        <joint name="$(arg robot_prefix)_joint1" value="0" />
+        <joint name="$(arg robot_prefix)_joint2" value="-0.785398163397" />
+        <joint name="$(arg robot_prefix)_joint3" value="0" />
+        <joint name="$(arg robot_prefix)_joint4" value="-2.35619449019" />
+        <joint name="$(arg robot_prefix)_joint5" value="0" />
+        <joint name="$(arg robot_prefix)_joint6" value="1.57079632679" />
+        <joint name="$(arg robot_prefix)_joint7" value="0.785398163397" />
     </group_state>
 </robot>

File: workspaces/franka/srdf/franka_dual_arm.srdf.xacro (robot description, xacro)
@@ -3,18 +3,13 @@
     <xacro:include filename="$(find franka_description)/robots/common/franka_arm.srdf.xacro"/>
     <xacro:franka_arm_srdf
-            arm_id="fr3_left"
+            robot_type="fr3"
             hand="false"
-            ee_id=""
             no_prefix="false"
-            arm_prefix=""
-            tip_link="link8"/>
-    <xacro:include filename="$(find franka_description)/robots/common/franka_arm.srdf.xacro"/>
+            arm_prefix="fr3_left"/>
     <xacro:franka_arm_srdf
-            arm_id="fr3_right"
+            robot_type="fr3"
             hand="false"
-            ee_id=""
             no_prefix="false"
-            arm_prefix=""
-            tip_link="link8"/>
+            arm_prefix="fr3_right"/>
     <group name="dual_arm">
         <group name="fr3_left_arm"/>

File: workspaces/franka/urdf/franka.urdf.xacro (robot description, xacro)
@@ -2,5 +2,5 @@
 <robot xmlns:xacro="http://www.ros.org/wiki/xacro" name="franka">
     <xacro:arg name="robot_type" default="fr3"/>
-    <xacro:arg name="arm_prefix" default="fr3"/>
+    <xacro:arg name="robot_prefix" default="fr3"/>
     <xacro:arg name="robot_ip" default="10.42.0.203"/>
     <xacro:arg name="ros2_control_hardware_type" default="mock"/>
@@ -20,5 +20,5 @@
                         dynamics="${xacro.load_yaml('$(find franka_description)/robots/fr3/dynamics.yaml')}"
                         hand="false"
-                        arm_prefix="$(arg arm_prefix)"
+                        arm_prefix="$(arg robot_prefix)"
                         ros2_control="true"
                         robot_ip="$(arg robot_ip)"
@@ -32,8 +32,8 @@
     </xacro:franka_robot>
     <!-- ============= TOOL MOUNT ================ -->
-    <link name="$(arg robot_type)_tool0"/>
-    <joint name="$(arg robot_type)_tool0_joint" type="fixed">
-        <parent link="$(arg robot_type)_link8"/>
-        <child link="$(arg robot_type)_tool0"/>
+    <link name="$(arg robot_prefix)_tool0"/>
+    <joint name="$(arg robot_prefix)_tool0_joint" type="fixed">
+        <parent link="$(arg robot_prefix)_link8"/>
+        <child link="$(arg robot_prefix)_tool0"/>
         <origin xyz="0 0 0" rpy="0 0 0"/>
     </joint>

File: workspaces/franka/urdf/franka_dual_arm.urdf.xacro (robot description, xacro)
@@ -1,16 +1,26 @@
 <?xml version="1.0"?>
 <robot xmlns:xacro="http://www.ros.org/wiki/xacro" name="franka_dual_arm">
-    <xacro:arg name="use_mock_hardware" default="true"/>
-    <xacro:arg name="robot_1_arm_id" default="fr3_left"/>
-    <xacro:arg name="robot_2_arm_id" default="fr3_right"/>
+    <!-- ============= ROBOT 1 (LEFT) ARGS ================ -->
+    <xacro:arg name="robot_1_ros2_control_hardware_type" default="mock"/>
+    <xacro:arg name="robot_1_prefix" default="fr3_left"/>
     <xacro:arg name="robot_1_ip" default="10.42.0.203"/>
-    <xacro:arg name="robot_1_scheduling_policy" default="detached"/>
+    <xacro:arg name="robot_1_mock_sensor_commands" default="true" />
+    <xacro:arg name="robot_1_is_async" default="true" />
+    <xacro:arg name="robot_1_scheduling_policy" default="slave" />
+    <xacro:arg name="robot_1_thread_priority" default="70" />
+    <xacro:arg name="robot_1_cpu_affinity" default="[2,3]" />
+    <!-- ============= ROBOT 2 (RIGHT) ARGS ================ -->
+    <xacro:arg name="robot_2_ros2_control_hardware_type" default="mock"/>
+    <xacro:arg name="robot_2_prefix" default="fr3_right"/>
     <xacro:arg name="robot_2_ip" default="10.42.0.204"/>
-    <xacro:arg name="robot_2_scheduling_policy" default="detached"/>
+    <xacro:arg name="robot_2_mock_sensor_commands" default="true" />
+    <xacro:arg name="robot_2_is_async" default="true" />
+    <xacro:arg name="robot_2_scheduling_policy" default="slave" />
+    <xacro:arg name="robot_2_thread_priority" default="70" />
+    <xacro:arg name="robot_2_cpu_affinity" default="[2,3]" />
     <link name="world"/>
+    <xacro:include filename="$(find franka_description)/robots/common/franka_robot.xacro"/>
     <!-- ============= FRANKA LEFT ================ -->
-    <xacro:include filename="$(find franka_description)/robots/common/franka_robot.xacro"/>
-    <xacro:franka_robot arm_id="$(arg robot_1_arm_id)"
-                        mesh_model="fr3"
+    <xacro:franka_robot robot_type="fr3"
                         joint_limits="${xacro.load_yaml('$(find franka_description)/robots/fr3/joint_limits.yaml')}"
                         inertials="${xacro.load_yaml('$(find franka_description)/robots/fr3/inertials.yaml')}"
@@ -18,24 +28,18 @@
                         dynamics="${xacro.load_yaml('$(find franka_description)/robots/fr3/dynamics.yaml')}"
                         hand="false"
-                        ee_id="franka_hand"
-                        safety_distance="0.03"
-                        xyz="0 -0.5 0"
-                        with_sc="false"
+                        arm_prefix="$(arg robot_1_prefix)"
                         ros2_control="true"
                         robot_ip="$(arg robot_1_ip)"
-                        use_fake_hardware="$(arg use_mock_hardware)"
-                        fake_sensor_commands="$(arg use_mock_hardware)"
-                        gazebo_effort="true"
-                        gazebo="false"
-                        no_prefix="false"
-                        arm_prefix=""
-                        description_pkg="franka_description"
+                        fake_sensor_commands="$(arg robot_1_mock_sensor_commands)"
                         connected_to="world"
-                        scheduling_policy="$(arg robot_1_scheduling_policy)">
+                        xyz="0 -0.5 0"
+                        ros2_control_hardware_type="$(arg robot_1_ros2_control_hardware_type)"
+                        is_async="$(arg robot_1_is_async)"
+                        scheduling_policy="$(arg robot_1_scheduling_policy)"
+                        thread_priority="$(arg robot_1_thread_priority)"
+                        cpu_affinity="$(arg robot_1_cpu_affinity)">
     </xacro:franka_robot>
     <!-- ============= FRANKA RIGHT ================ -->
-    <xacro:include filename="$(find franka_description)/robots/common/franka_robot.xacro"/>
-    <xacro:franka_robot arm_id="$(arg robot_2_arm_id)"
-                        mesh_model="fr3"
+    <xacro:franka_robot robot_type="fr3"
                         joint_limits="${xacro.load_yaml('$(find franka_description)/robots/fr3/joint_limits.yaml')}"
                         inertials="${xacro.load_yaml('$(find franka_description)/robots/fr3/inertials.yaml')}"
@@ -43,32 +47,28 @@
                         dynamics="${xacro.load_yaml('$(find franka_description)/robots/fr3/dynamics.yaml')}"
                         hand="false"
-                        ee_id="franka_hand"
-                        safety_distance="0.03"
-                        xyz="0 0.5 0"
-                        with_sc="false"
+                        arm_prefix="$(arg robot_2_prefix)"
                         ros2_control="true"
                         robot_ip="$(arg robot_2_ip)"
-                        use_fake_hardware="$(arg use_mock_hardware)"
-                        fake_sensor_commands="$(arg use_mock_hardware)"
-                        gazebo_effort="true"
-                        gazebo="false"
-                        no_prefix="false"
-                        arm_prefix=""
-                        description_pkg="franka_description"
+                        fake_sensor_commands="$(arg robot_2_mock_sensor_commands)"
                         connected_to="world"
-                        scheduling_policy="$(arg robot_2_scheduling_policy)">
+                        xyz="0 0.5 0"
+                        ros2_control_hardware_type="$(arg robot_2_ros2_control_hardware_type)"
+                        is_async="$(arg robot_2_is_async)"
+                        scheduling_policy="$(arg robot_2_scheduling_policy)"
+                        thread_priority="$(arg robot_2_thread_priority)"
+                        cpu_affinity="$(arg robot_2_cpu_affinity)">
     </xacro:franka_robot>
     <!-- ============= FRANKA LEFT TOOL MOUNT ================ -->
-    <link name="$(arg robot_1_arm_id)_tool0"/>
-    <joint name="$(arg robot_1_arm_id)_tool0_joint" type="fixed">
-        <parent link="$(arg robot_1_arm_id)_link8"/>
-        <child link="$(arg robot_1_arm_id)_tool0"/>
+    <link name="$(arg robot_1_prefix)_tool0"/>
+    <joint name="$(arg robot_1_prefix)_tool0_joint" type="fixed">
+        <parent link="$(arg robot_1_prefix)_link8"/>
+        <child link="$(arg robot_1_prefix)_tool0"/>
         <origin xyz="0 0 0" rpy="0 0 0"/>
     </joint>
     <!-- ============= FRANKA RIGHT TOOL MOUNT ================ -->
-    <link name="$(arg robot_2_arm_id)_tool0"/>
-    <joint name="$(arg robot_2_arm_id)_tool0_joint" type="fixed">
-        <parent link="$(arg robot_2_arm_id)_link8"/>
-        <child link="$(arg robot_2_arm_id)_tool0"/>
+    <link name="$(arg robot_2_prefix)_tool0"/>
+    <joint name="$(arg robot_2_prefix)_tool0_joint" type="fixed">
+        <parent link="$(arg robot_2_prefix)_link8"/>
+        <child link="$(arg robot_2_prefix)_tool0"/>
         <origin xyz="0 0 0" rpy="0 0 0"/>
     </joint>
