Commit message: update franka description, add foreman and moveit trajectory smoothing plugin

File: workspaces/franka/urdf/franka.urdf.xacro (robot description, xacro)
@@ -1,12 +1,18 @@
 <?xml version="1.0"?>
 <robot xmlns:xacro="http://www.ros.org/wiki/xacro" name="franka">
-    <xacro:arg name="use_mock_hardware" default="true"/>
-    <xacro:arg name="arm_id" default="fr3"/>
+    <xacro:arg name="robot_type" default="fr3"/>
+    <xacro:arg name="arm_prefix" default="fr3"/>
     <xacro:arg name="robot_ip" default="10.42.0.203"/>
-    <xacro:arg name="scheduling_policy" default="detached"/>
+    <xacro:arg name="ros2_control_hardware_type" default="mock"/>
+    <xacro:property name="ros2_control_hardware_type" value="$(arg ros2_control_hardware_type)"/>
+    <xacro:arg name="mock_sensor_commands" default="true" />
+    <xacro:arg name="is_async" default="true" />
+    <xacro:arg name="scheduling_policy" default="slave" />
+    <xacro:arg name="thread_priority" default="70" />
+    <xacro:arg name="cpu_affinity" default="[2,3]" />
     <link name="world"/>
     <!-- ============= FRANKA ================ -->
     <xacro:include filename="$(find franka_description)/robots/common/franka_robot.xacro"/>
-    <xacro:franka_robot arm_id="$(arg arm_id)"
+    <xacro:franka_robot robot_type="$(arg robot_type)"
                         joint_limits="${xacro.load_yaml('$(find franka_description)/robots/fr3/joint_limits.yaml')}"
                         inertials="${xacro.load_yaml('$(find franka_description)/robots/fr3/inertials.yaml')}"
@@ -14,24 +20,20 @@
                         dynamics="${xacro.load_yaml('$(find franka_description)/robots/fr3/dynamics.yaml')}"
                         hand="false"
-                        ee_id="franka_hand"
-                        safety_distance="0.03"
-                        with_sc="false"
+                        arm_prefix="$(arg arm_prefix)"
                         ros2_control="true"
                         robot_ip="$(arg robot_ip)"
-                        use_fake_hardware="$(arg use_mock_hardware)"
-                        fake_sensor_commands="$(arg use_mock_hardware)"
-                        gazebo_effort="true"
-                        gazebo="false"
-                        no_prefix="false"
-                        arm_prefix=""
-                        description_pkg="franka_description"
+                        fake_sensor_commands="$(arg mock_sensor_commands)"
                         connected_to="world"
-                        scheduling_policy="$(arg scheduling_policy)">
+                        ros2_control_hardware_type="${ros2_control_hardware_type}"
+                        is_async="$(arg is_async)"
+                        scheduling_policy="$(arg scheduling_policy)"
+                        thread_priority="$(arg thread_priority)"
+                        cpu_affinity="$(arg cpu_affinity)">
     </xacro:franka_robot>
     <!-- ============= TOOL MOUNT ================ -->
-    <link name="$(arg arm_id)_tool0"/>
-    <joint name="$(arg arm_id)_tool0_joint" type="fixed">
-        <parent link="$(arg arm_id)_link8"/>
-        <child link="$(arg arm_id)_tool0"/>
+    <link name="$(arg robot_type)_tool0"/>
+    <joint name="$(arg robot_type)_tool0_joint" type="fixed">
+        <parent link="$(arg robot_type)_link8"/>
+        <child link="$(arg robot_type)_tool0"/>
         <origin xyz="0 0 0" rpy="0 0 0"/>
     </joint>

Commit message: Update franka workspace (#14)
* update franka description, add foreman and moveit trajectory smoothing plugin

* add foreman, update launch files

File: workspaces/franka/urdf/franka.urdf.xacro (robot description, xacro)
@@ -1,12 +1,18 @@
 <?xml version="1.0"?>
 <robot xmlns:xacro="http://www.ros.org/wiki/xacro" name="franka">
-    <xacro:arg name="use_mock_hardware" default="true"/>
-    <xacro:arg name="arm_id" default="fr3"/>
+    <xacro:arg name="robot_type" default="fr3"/>
+    <xacro:arg name="robot_prefix" default="fr3"/>
     <xacro:arg name="robot_ip" default="10.42.0.203"/>
-    <xacro:arg name="scheduling_policy" default="detached"/>
+    <xacro:arg name="ros2_control_hardware_type" default="mock"/>
+    <xacro:property name="ros2_control_hardware_type" value="$(arg ros2_control_hardware_type)"/>
+    <xacro:arg name="mock_sensor_commands" default="true" />
+    <xacro:arg name="is_async" default="true" />
+    <xacro:arg name="scheduling_policy" default="slave" />
+    <xacro:arg name="thread_priority" default="70" />
+    <xacro:arg name="cpu_affinity" default="[2,3]" />
     <link name="world"/>
     <!-- ============= FRANKA ================ -->
     <xacro:include filename="$(find franka_description)/robots/common/franka_robot.xacro"/>
-    <xacro:franka_robot arm_id="$(arg arm_id)"
+    <xacro:franka_robot robot_type="$(arg robot_type)"
                         joint_limits="${xacro.load_yaml('$(find franka_description)/robots/fr3/joint_limits.yaml')}"
                         inertials="${xacro.load_yaml('$(find franka_description)/robots/fr3/inertials.yaml')}"
@@ -14,24 +20,20 @@
                         dynamics="${xacro.load_yaml('$(find franka_description)/robots/fr3/dynamics.yaml')}"
                         hand="false"
-                        ee_id="franka_hand"
-                        safety_distance="0.03"
-                        with_sc="false"
+                        arm_prefix="$(arg robot_prefix)"
                         ros2_control="true"
                         robot_ip="$(arg robot_ip)"
-                        use_fake_hardware="$(arg use_mock_hardware)"
-                        fake_sensor_commands="$(arg use_mock_hardware)"
-                        gazebo_effort="true"
-                        gazebo="false"
-                        no_prefix="false"
-                        arm_prefix=""
-                        description_pkg="franka_description"
+                        fake_sensor_commands="$(arg mock_sensor_commands)"
                         connected_to="world"
-                        scheduling_policy="$(arg scheduling_policy)">
+                        ros2_control_hardware_type="${ros2_control_hardware_type}"
+                        is_async="$(arg is_async)"
+                        scheduling_policy="$(arg scheduling_policy)"
+                        thread_priority="$(arg thread_priority)"
+                        cpu_affinity="$(arg cpu_affinity)">
     </xacro:franka_robot>
     <!-- ============= TOOL MOUNT ================ -->
-    <link name="$(arg arm_id)_tool0"/>
-    <joint name="$(arg arm_id)_tool0_joint" type="fixed">
-        <parent link="$(arg arm_id)_link8"/>
-        <child link="$(arg arm_id)_tool0"/>
+    <link name="$(arg robot_prefix)_tool0"/>
+    <joint name="$(arg robot_prefix)_tool0_joint" type="fixed">
+        <parent link="$(arg robot_prefix)_link8"/>
+        <child link="$(arg robot_prefix)_tool0"/>
         <origin xyz="0 0 0" rpy="0 0 0"/>
     </joint>
